File: Swadge-S2-Devkit/Swadge-S2-Devkit.kicad_pcb (KiCad board)
At the start: 2 copper layers, 134 x 100 mm, 102 parts, among them J1 CurrentMonitor, J2 DEBUG_BANK_C, J3 DEBUG_BANK_B, J4 DEBUG_BANK_A, J5 MICSEL, J6 TRYMIC, J7 LEDK_J, J8 LCD18, J9 LCD28, M1 VZ43FC1B5640007L, P1 USB_C_Plug_USB2.0, Q1 Q_N_FET, Q2 AP2003_PN_FET, Q3 AP2003_PN_FET, Q4 AP2003_PN_FET, SW1 4-1437565-2, SW10 BLISTER_SILICONE_BUTTON, SW11 touch-ring-6, SW14 SW_SPDT, SW2 4-1437565-2, SW3 4-1437565-2, SW4 4-1437565-2, SW5 4-1437565-2, SW6 4-1437565-2, SW7 4-1437565-2, SW8 4-1437565-2, SW9 4-1437565-2, U1 ESP32-S2-SOLO, U10 GENERIC_LDO_2.8, U11 LCD_240x240_1.3_12, U12 LCD_135x240_1.14_13, U15 LCD_240x240_1.54_12, U2 BUS_PCIexpress, U3 MT3410, U4 GS321-TR, U5 QMA7981, U6 INGHAi_GSPK2308P-8R0.5W, U9 GENERIC_LDO_1.8

Commit message: Messing around with another party ball
Parts:
- removed Ref**: Val**, Swadge_Parts:swadges-family
- removed svg2mod: G***, Swadge_Parts:MAGFEST_logo_centered_final
- added G*** (x6): LOGO, LOGO, F.Cu at (150.0, 100.0)
- BT1, BT2, BT3, C1, C10, C11, C15, C17, C2, C3, C8, C9, D7, L1, L2, Q1, Q2, Q3, Q4, R1, R10, R15, R16, R17, R18, R19, R20, R23, R26, R5, R6, R7, R8, R9, U11, U12, U15, U2, U4: moved to F.Cu
- moved U15 217.0 mm to (2.58, 33.7), turned to 0 degrees
- moved U12 210.1 mm to (25.8, 33.7), turned to 0 degrees
- moved J9 206.5 mm to (37.5, 28.5)
- moved J8 196.9 mm to (37.5, 38.2)
- moved M1 192.9 mm to (-10.4, 81.9), turned to 0 degrees
- moved U2 191.3 mm to (-14.8, 74.5), turned to 0 degrees
- moved J5 191.0 mm to (-0.85, 81.4)
- moved C11 189.7 mm to (3.48, 87.9), turned to 0 degrees
- moved D7 189.5 mm to (-12.3, 87.0), turned to 0 degrees
- moved U11 175.5 mm to (56.1, 18.2), turned to 0 degrees
- moved BT2 170.0 mm to (12.8, 17.1), turned to 0 degrees
- moved L2 166.6 mm to (52.1, 87.3), turned to 0 degrees
- moved SW2 161.7 mm to (30.0, 83.4), turned to 0 degrees
- moved R20 156.2 mm to (3.48, 80.4), turned to 0 degrees
- moved J7 153.0 mm to (84.6, 38.1), turned to 0 degrees
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Routing:
- net GND: track 772.3 -> 0.00 mm, vias 122 -> 0
- net +3V3: track 458.2 -> 0.00 mm, vias 18 -> 0
- net BTN_8: track 144.2 -> 0.00 mm, vias 4 -> 0
- net BTN_2: track 124.1 -> 0.00 mm, vias 2 -> 0
- net TFT_RS: track 122.8 -> 0.00 mm, vias 6 -> 0
- net BTN_3: track 114.9 -> 0.00 mm, vias 4 -> 0
- net TX: track 112.8 -> 0.00 mm, vias 2 -> 0
- net LED: track 112.4 -> 0.00 mm, vias 4 -> 0
- net RX: track 110.6 -> 0.00 mm, vias 2 -> 0
- net BTN_5: track 107.9 -> 0.00 mm, vias 2 -> 0
- net TFT_CS: track 107.7 -> 0.00 mm, vias 4 -> 0
- net BLISTER1: track 103.2 -> 0.00 mm, vias 4 -> 0
- net BTN_4: track 102.7 -> 0.00 mm, vias 3 -> 0
- net TFT_RESET: track 99.7 -> 0.00 mm, vias 2 -> 0
- net TFT_SCL: track 97.2 -> 0.00 mm, vias 2 -> 0
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- removed copper zone on B.Cu, net GND
- removed copper zone on F.Cu, net GND
Other:
- board size 134 x 100 mm -> 94.6 x 100 mm
- rule pad_to_mask_clearance: 0 -> 0.2
- board text removed: "+ -"
- board text removed: "Swadge S2 Devkit 1.0.0"
